File: kicad/thyme.kicad_pcb (KiCad board)
At the start: 2 copper layers, 18.3 x 33.6 mm, 86 parts, among them SW1 SW_Push, SW10 SW_Push, SW11 SW_Push, SW12 SW_Push, SW13 SW_Push, SW14 SW_Push, SW15 SW_Push, SW16 SW_Push, SW17 SW_Push, SW18 SW_Push, SW19 SW_Push, SW2 SW_Push, SW20 SW_Push, SW21 SW_Push, SW22 SW_Push, SW23 SW_Push, SW24 SW_Push, SW25 SW_Push, SW26 SW_Push, SW27 SW_Push, SW28 SW_Push, SW29 SW_Push, SW3 SW_Push, SW30 SW_Push, SW31 SW_Push, SW32 SW_Push, SW33 SW_Push, SW34 SW_Push, SW35 SW_Push, SW36 SW_Push, SW37 SW_Push, SW38 SW_Push, SW39 SW_Push, SW4 SW_Push, SW40 SW_Push, SW41 SW_Push, SW42 SW_Push, SW5 SW_Push, SW6 SW_Push, SW7 SW_Push, SW8 SW_Push, SW9 SW_Push, U1 nice_nano, U2 nice_nano

Commit message: bug: fix row 5 being unconnected
Parts:
- added J1: JST BATTERY, Connector_JST:JST_PH_B2B-PH-K_1x02_P2.00mm_Vertical, F.Cu at (122.6, 114.8)
- added J2: JST BATTERY, Connector_JST:JST_PH_B2B-PH-K_1x02_P2.00mm_Vertical, F.Cu at (122.6, 121.3)
- added SW44: SW_SPDT, Button_Switch_THT:SW_Slide-03_Wuerth-WS-SLTV_10x2.5x6.4_P2.54mm, F.Cu at (133.4, 114.1)
- added SW45: SW_SPDT, Button_Switch_THT:SW_Slide-03_Wuerth-WS-SLTV_10x2.5x6.4_P2.54mm, F.Cu at (133.4, 118.1)
- moved D28 26.2 mm to (60.6, 131.6)
- moved D33 26.2 mm to (60.6, 149.3)
- moved D11 26.2 mm to (39.1, 149.3)
- moved D39 26.2 mm to (71.4, 131.6)
- moved D6 26.2 mm to (39.1, 131.6)
- moved D17 26.2 mm to (49.9, 131.6)
- moved D22 26.2 mm to (49.9, 149.3)
- moved D23 26.2 mm to (60.6, 113.8)
- moved D25 26.2 mm to (60.6, 120.9)
- moved D1 26.2 mm to (39.1, 113.8)
- moved D24 26.2 mm to (60.6, 117.4)
- moved D27 26.2 mm to (60.6, 128.0)
- moved D29 26.2 mm to (60.6, 135.1)
- moved D3 26.2 mm to (39.1, 120.9)
- moved D30 26.2 mm to (60.6, 138.7)
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Connections:
- SW16 pad 2: unconnected-(SW16-Pad2) -> L-COL5
- SW17 pad 2: unconnected-(SW17-Pad2) -> L-COL5
- SW18 pad 2: unconnected-(SW18-Pad2) -> L-COL5
- SW19 pad 2: L-COL5 -> L-COL6
- SW20 pad 2: L-COL5 -> L-COL6
- SW21 pad 2: L-COL5 -> L-COL6
- SW37 pad 2: unconnected-(SW37-Pad2) -> R-COL5
- SW38 pad 2: unconnected-(SW38-Pad2) -> R-COL5
- SW39 pad 2: unconnected-(SW39-Pad2) -> R-COL5
- SW40 pad 2: R-COL5 -> R-COL6
- SW41 pad 2: R-COL5 -> R-COL6
- SW42 pad 2: R-COL5 -> R-COL6
- U1 pad 1: unconnected-(U1-P0.06-Pad1) -> L-ROW0
- U1 pad 10: unconnected-(U1-P0.11-Pad10) -> L-COL4
- U1 pad 11: unconnected-(U1-P1.04-LF-Pad11) -> L-COL5
- U1 pad 12: unconnected-(U1-P1.06-LF-Pad12) -> L-COL6
- U1 pad 2: unconnected-(U1-P0.08-Pad2) -> L-ROW1
- U1 pad 29: unconnected-(U1-BAT+-Pad29) -> Net-(SW44-B)
- U1 pad 5: unconnected-(U1-P0.17-Pad5) -> L-ROW2
- U1 pad 6: unconnected-(U1-P0.20-Pad6) -> L-COL0
- U1 pad 7: unconnected-(U1-P0.22-Pad7) -> L-COL1
- U1 pad 8: unconnected-(U1-P0.24-Pad8) -> L-COL2
- U1 pad 9: unconnected-(U1-P1.00-Pad9) -> L-COL3
- U2 pad 1: unconnected-(U2-P0.06-Pad1) -> R-ROW0
- U2 pad 10: unconnected-(U2-P0.11-Pad10) -> R-COL4
- U2 pad 11: unconnected-(U2-P1.04-LF-Pad11) -> R-COL5
- U2 pad 12: unconnected-(U2-P1.06-LF-Pad12) -> R-COL6
- U2 pad 2: unconnected-(U2-P0.08-Pad2) -> R-ROW1
- U2 pad 29: unconnected-(U2-BAT+-Pad29) -> Net-(SW45-B)
- U2 pad 5: unconnected-(U2-P0.17-Pad5) -> R-ROW2
- U2 pad 6: unconnected-(U2-P0.20-Pad6) -> R-COL0
- U2 pad 7: unconnected-(U2-P0.22-Pad7) -> R-COL1
- U2 pad 8: unconnected-(U2-P0.24-Pad8) -> R-COL2
- U2 pad 9: unconnected-(U2-P1.00-Pad9) -> R-COL3

Commit message: chore: split power into left and right and add no connects
Parts:
- moved D19 172.2 mm to (107.2, -23.7)
- moved D30 172.2 mm to (118.0, -23.7)
- moved D41 172.2 mm to (128.7, -23.7)
- moved D8 172.2 mm to (96.4, -23.7)
- moved SW1 172.2 mm to (103.1, -141.4)
- moved SW13 172.2 mm to (136.2, -141.4)
- moved SW19 172.2 mm to (152.8, -141.4)
- moved SW25 172.2 mm to (169.3, -141.4)
- moved SW31 172.2 mm to (185.9, -141.4)
- moved SW37 172.2 mm to (202.4, -141.4)
- moved SW7 172.2 mm to (119.7, -141.4)
- moved D1 172.2 mm to (96.4, -48.6)
- moved D10 172.2 mm to (96.4, -16.6)
- moved D11 172.2 mm to (96.4, -13.1)
- moved D12 172.2 mm to (107.2, -48.6)
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Connections:
- J1 pad 1: BATTERY_POSITIVE -> LBATTERY_POSITIVE
- J1 pad 2: BATTERY_NEGATIVE -> LPOWER-GND
- J2 pad 1: BATTERY_POSITIVE -> RBATTERY_POSITIVE
- J2 pad 2: BATTERY_NEGATIVE -> RPOWER-GND
- SW44 pad 2: GND -> LBATTERY_POSITIVE
- SW44 pad 3: BATTERY_POSITIVE -> unconnected-(SW44-A-Pad3)
- SW45 pad 2: GND -> RBATTERY_POSITIVE
- SW45 pad 3: BATTERY_POSITIVE -> unconnected-(SW45-A-Pad3)
- U1 pad 1: L-ROW0 -> unconnected-(U1-P0.06-Pad1)
- U1 pad 14: GND -> LPOWER-GND
- U1 pad 16: +3.3V -> LPOWER-3.3V
- U1 pad 17: unconnected-(U1-P0.31-LF-Pad17) -> L-ROW0
- U1 pad 18: unconnected-(U1-P0.29-LF-Pad18) -> L-ROW1
- U1 pad 2: L-ROW1 -> unconnected-(U1-P0.08-Pad2)_1
- U1 pad 28: GND -> LPOWER-GND
- U1 pad 3: GND -> LPOWER-GND
- U1 pad 4: GND -> LPOWER-GND
- U2 pad 1: R-ROW0 -> unconnected-(U2-P0.06-Pad1)_1
- U2 pad 14: GND -> RPOWER-GND
- U2 pad 16: +3.3V -> RPOWER-3.3V
- U2 pad 17: unconnected-(U2-P0.31-LF-Pad17) -> R-ROW0
- U2 pad 18: unconnected-(U2-P0.29-LF-Pad18) -> R-ROW1
- U2 pad 2: R-ROW1 -> unconnected-(U2-P0.08-Pad2)_1
- U2 pad 28: GND -> RPOWER-GND
- U2 pad 3: GND -> RPOWER-GND
- U2 pad 4: GND -> RPOWER-GND

Commit message: chore: move around footprints
Parts:
- moved D34 248.2 mm to (347.9, 68.0)
- moved D35 248.2 mm to (347.9, 71.5)
- moved D36 248.2 mm to (347.9, 75.0)
- moved D37 248.2 mm to (347.9, 78.6)
- moved D38 248.2 mm to (347.9, 82.2)
- moved D39 248.2 mm to (347.9, 85.7)
- moved D40 248.2 mm to (347.9, 89.2)
- moved D41 248.2 mm to (347.9, 92.8)
- moved D42 248.2 mm to (347.9, 96.3)
- moved D23 246.5 mm to (337.1, 64.4)
- moved D24 246.5 mm to (337.1, 67.9)
- moved D25 246.5 mm to (337.1, 71.5)
- moved D26 246.5 mm to (337.1, 75.0)
- moved D27 246.5 mm to (337.1, 78.6)
- moved D28 246.5 mm to (337.1, 82.1)
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
Commit message: feat: align key switches in pcb
Parts:
- moved SW40 88.6 mm to (165.5, 96.8)
- moved SW22 85.6 mm to (273.5, 45.9)
- moved SW23 85.3 mm to (273.5, 62.9)
- moved SW24 85.0 mm to (273.5, 79.8)
- moved SW41 72.4 mm to (183.5, 96.8)
- moved SW37 70.6 mm to (183.5, 45.9)
- moved SW38 70.6 mm to (183.5, 62.9)
- moved SW39 70.6 mm to (183.5, 79.8)
- moved SW34 62.1 mm to (201.5, 45.9)
- moved SW42 61.9 mm to (201.5, 96.8)
- moved SW35 61.7 mm to (201.5, 62.9)
- moved SW36 61.4 mm to (201.5, 79.8)
- moved SW19 61.2 mm to (131.8, 96.8)
- moved SW16 60.8 mm to (113.8, 45.9)
- moved SW17 60.4 mm to (113.8, 62.9)
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
Commit message: feat: arrange switches and add edge cuts
Parts:
- J1, J2: footprint Connector_JST:JST_PH_B2B-PH-K_1x02_P2.00mm_Vertical -> Connector_JST:JST_PH_S2B-PH-SM4-TB_1x02-1MP_P2.00mm_Horizontal
- moved SW21 9.86 mm to (87.1, 101.6)
- moved J1 9.63 mm to (129.4, 83.8), turned to 90 degrees
- moved J2 9.45 mm to (168.2, 83.8), turned to -90 degrees
- moved SW42 9.10 mm to (209.2, 101.6)
- moved SW24 8.90 mm to (278.2, 87.4)
- moved SW3 8.90 mm to (19.0, 87.4)
- moved SW20 8.76 mm to (108.7, 104.0), turned to -15 degrees
- moved SW27 8.41 mm to (259.2, 87.4)
- moved SW6 8.41 mm to (38.0, 87.4)
- moved SW41 8.25 mm to (187.6, 104.0), turned to 15 degrees
- moved SW2 7.29 mm to (19.0, 68.4)
- moved SW23 7.29 mm to (278.2, 68.4)
- moved SW26 6.68 mm to (259.2, 68.4)
- moved SW5 6.68 mm to (38.0, 68.4)
- moved SW1 5.92 mm to (19.0, 49.4)
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Other:
- board size 18.3 x 33.6 mm -> 280.6 x 83.1 mm

Commit message: feat: place diodes
Parts:
- moved D19 307.4 mm to (287.8, 53.2), turned to 90 degrees
- moved D21 307.2 mm to (287.8, 92.4), turned to 90 degrees
- moved D20 306.9 mm to (287.8, 72.2), turned to 90 degrees
- moved D39 252.0 mm to (96.6, 105.4), turned to 90 degrees
- moved D38 229.8 mm to (119.0, 102.9), turned to -105 degrees
- moved D37 207.1 mm to (141.4, 95.2), turned to 150 degrees
- moved D40 191.8 mm to (156.2, 95.2), turned to 30 degrees
- moved D34 156.1 mm to (192.8, 50.8), turned to 90 degrees
- moved D36 155.7 mm to (192.8, 88.8), turned to 90 degrees
- moved D35 155.1 mm to (192.8, 69.8), turned to 90 degrees
- moved D41 150.6 mm to (197.8, 105.0), turned to 105 degrees
- moved D18 144.6 mm to (123.9, 89.1), turned to 90 degrees
- moved D17 143.1 mm to (123.9, 69.8), turned to 90 degrees
- moved D16 143.0 mm to (123.5, 50.8), turned to 90 degrees
- moved D31 133.0 mm to (211.8, 48.4), turned to 90 degrees
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Other:
- board size 280.6 x 83.1 mm -> 281.8 x 83.1 mm

Commit message: feat: add new jst connector and route the board
Parts:
- removed J1, J2: JST BATTERY, Connector_JST:JST_PH_S2B-PH-SM4-TB_1x02-1MP_P2.00mm_Horizontal
- added P1: JST BATTERY L, libraries:JST_S2B-PH-SM4-TB, F.Cu at (125.4, 84.1)
- added P2: JST BATTERY R, libraries:JST_S2B-PH-SM4-TB, F.Cu at (171.9, 83.8)
- moved D18 14.9 mm to (117.8, 75.5), turned to 180 degrees
- moved D37 7.25 mm to (135.1, 91.7), turned to -30 degrees
- moved D28 1.96 mm to (230.7, 48.3)
Connections:
- U1 pad 10: L-COL4 -> L-COL2
- U1 pad 11: L-COL5 -> L-ROW2
- U1 pad 12: L-COL6 -> L-ROW1
- U1 pad 13: unconnected-(U1-BAT+-Pad13) -> Net-(SW44-B)
- U1 pad 18: L-ROW1 -> unconnected-(U1-P0.29-LF-Pad18)
- U1 pad 29: Net-(SW44-B) -> unconnected-(U1-BAT+-Pad29)
- U1 pad 5: L-ROW2 -> L-COL0
- U1 pad 6: L-COL0 -> L-COL1
- U1 pad 7: L-COL1 -> L-COL3
- U1 pad 8: L-COL2 -> L-COL4
- U1 pad 9: L-COL3 -> L-COL5
- U2 pad 10: R-COL4 -> R-ROW2
- U2 pad 11: R-COL5 -> unconnected-(U2-P1.04-LF-Pad11)
- U2 pad 13: unconnected-(U2-BAT+-Pad13) -> Net-(SW45-B)
- U2 pad 18: R-ROW1 -> R-COL0
- U2 pad 19: unconnected-(U2-P0.02-LF-Pad19) -> R-COL1
- U2 pad 20: unconnected-(U2-P1.15-LF-Pad20) -> R-COL2
- U2 pad 21: unconnected-(U2-P1.13-LF-Pad21) -> R-COL3
- U2 pad 22: unconnected-(U2-P1.11-LF-Pad22) -> R-COL4
- U2 pad 23: unconnected-(U2-P0.10-LF-Pad23) -> R-COL5
- U2 pad 24: unconnected-(U2-P0.09-LF-Pad24) -> R-ROW1
- U2 pad 29: Net-(SW45-B) -> unconnected-(U2-BAT+-Pad29)
- U2 pad 5: R-ROW2 -> unconnected-(U2-P0.17-Pad5)
- U2 pad 6: R-COL0 -> unconnected-(U2-P0.20-Pad6)
- U2 pad 7: R-COL1 -> unconnected-(U2-P0.22-Pad7)
- U2 pad 8: R-COL2 -> unconnected-(U2-P0.24-Pad8)
- U2 pad 9: R-COL3 -> unconnected-(U2-P1.00-Pad9)
Routing:
- net R-ROW0: track 0.00 -> 186.9 mm
- net R-ROW2: track 0.00 -> 174.3 mm
- net L-ROW0: track 0.00 -> 169.3 mm
- net R-COL0: track 0.00 -> 162.8 mm
- net R-ROW1: track 0.00 -> 161.6 mm
- net L-COL0: track 0.00 -> 152.0 mm, vias 0 -> 1
- net R-COL1: track 0.00 -> 143.0 mm
- net L-ROW1: track 0.00 -> 140.8 mm
- net L-ROW2: track 0.00 -> 137.5 mm, vias 0 -> 1
- net L-COL1: track 0.00 -> 130.1 mm, vias 0 -> 2
- net R-COL2: track 0.00 -> 121.8 mm
- net L-COL2: track 0.00 -> 111.1 mm
- net R-COL3: track 0.00 -> 98.9 mm
- net L-COL3: track 0.00 -> 89.0 mm
- net R-COL6: track 0.00 -> 87.4 mm
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- added copper zone on B.Cu, net LPOWER-GND
- added copper zone on B.Cu, net RPOWER-GND
Other:
- outline, holes or cut-outs redrawn
