File: kicad/panelization/panelized.kicad_pcb (KiCad board)
At the start: 2 copper layers, 301.4 x 102.3 mm, 187 parts, among them J1 JST BATTERY R, J2 JST BATTERY R, SW1 SW_Push, SW10 SW_Push, SW11 SW_Push, SW12 SW_Push, SW13 SW_Push, SW14 SW_Push, SW15 SW_Push, SW16 SW_Push, SW17 SW_Push, SW18 SW_Push, SW19 SW_Push, SW2 SW_Push, SW20 SW_Push, SW21 SW_Push, SW22 SW_Push, SW23 SW_Push, SW24 SW_Push, SW25 SW_Push, SW26 SW_Push, SW27 SW_Push, SW28 SW_Push, SW29 SW_Push, SW3 SW_Push, SW30 SW_Push, SW31 SW_Push, SW32 SW_Push, SW33 SW_Push, SW34 SW_Push, SW35 SW_Push, SW36 SW_Push, SW37 SW_Push, SW38 SW_Push, SW39 SW_Push, SW4 SW_Push, SW40 SW_Push, SW41 SW_Push, SW42 SW_Push, SW5 SW_Push, SW6 SW_Push, SW7 SW_Push, SW8 SW_Push, SW9 SW_Push, U1 nice_nano, U2 nice_nano

Commit message: feat: move to 6 connectors and remove silkscreen lables
Parts:
- removed the KiKit_MB_10_1 at (93.2, 102.9)
- removed KiKit_MB_12_6, KiKit_MB_12_7, KiKit_MB_13_1, KiKit_MB_13_2, KiKit_MB_13_3, KiKit_MB_13_4, KiKit_MB_13_5, KiKit_MB_13_6, KiKit_MB_13_7, KiKit_MB_14_1, KiKit_MB_14_2, KiKit_MB_14_3, KiKit_MB_14_4, KiKit_MB_14_5, KiKit_MB_15_1, KiKit_MB_15_2, KiKit_MB_15_3, KiKit_MB_15_4, KiKit_MB_15_5, KiKit_MB_15_6, KiKit_MB_15_7, KiKit_MB_16_1, KiKit_MB_16_2, KiKit_MB_16_3, KiKit_MB_16_4, KiKit_MB_16_5: NPTH, NPTH
- added ?: , , F.Cu at (198.8, 113.3)
- added ?: , , F.Cu at (151.2, 112.8)
- added ?: , , F.Cu at (199.2, 113.9)
- added ?: , , F.Cu at (150.8, 113.4)
- added KiKit_MB_10_1: NPTH, NPTH, F.Cu at (199.2, 113.9)
- added KiKit_MB_10_1: NPTH, NPTH, F.Cu at (198.8, 113.3)
- added KiKit_MB_10_1: NPTH, NPTH, F.Cu at (198.5, 112.5)
- added KiKit_MB_9_6: NPTH, NPTH, F.Cu at (152.1, 111.1)
- added KiKit_MB_9_7: NPTH, NPTH, F.Cu at (151.5, 112.1)
- added KiKit_MB_9_7: NPTH, NPTH, F.Cu at (151.2, 112.8)
- added KiKit_MB_9_7: NPTH, NPTH, F.Cu at (150.8, 113.4)
- moved KiKit_MB_7_5 205.3 mm to (65.3, 91.8)
- moved KiKit_MB_7_4 203.4 mm to (66.3, 91.8)
- moved KiKit_MB_7_3 201.5 mm to (67.3, 91.8)
- moved KiKit_MB_7_2 199.7 mm to (68.3, 91.8)
- moved KiKit_MB_8_5 198.8 mm to (108.4, 106.1)
- moved KiKit_MB_7_1 197.8 mm to (69.3, 91.8)
- moved KiKit_MB_8_4 196.9 mm to (109.4, 106.1)
- moved KiKit_MB_8_3 195.0 mm to (110.4, 106.1)
- moved KiKit_MB_8_2 193.2 mm to (111.4, 106.1)
- moved KiKit_MB_8_1 191.3 mm to (112.4, 106.1)
- moved KiKit_MB_12_1 124.9 mm to (284.7, 92.2)
- moved KiKit_MB_12_2 124.6 mm to (283.7, 92.2)
- moved KiKit_MB_12_3 124.2 mm to (282.7, 92.2)
- moved KiKit_MB_12_4 123.9 mm to (281.7, 92.2)
- moved KiKit_MB_12_5 123.5 mm to (280.7, 92.2)
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Other:
- outline, holes or cut-outs redrawn
- board text added: ""THYME v1.18""
- board text added: "Created on 2025-11-12 JLC Order: JLCJLCJLC"
- board text added: "topside"
- board text removed: ""THYME v1.19-jlc""
- board text removed: "Created on 2025-05-03 PCBWAY Order: WAYWAYWAY"
